Commit message: Imported upstream version '0.2.5' of 'upstream'

File: urdf/02-multipleshapes.urdf (robot description, URDF)
Before this commit: robot multipleshapes, 2 links, 1 joints
Links:
- link right_leg: geometry visual box size=0.6 0.1 0.2

File: urdf/03-origins.urdf (robot description, URDF)
Before this commit: robot origins, 2 links, 1 joints
Links:
- link right_leg: geometry visual box size=0.6 0.1 0.2
Joints:
- joint base_to_right_leg: origin xyz=0.22 0 .25 -> xyz=0 -0.22 0.25

File: urdf/04-materials.urdf (robot description, URDF)
Before this commit: robot materials, 3 links, 2 joints
Links:
- link left_leg: geometry visual box size=0.6 0.1 0.2
- link right_leg: geometry visual box size=0.6 0.1 0.2
Joints:
- joint base_to_left_leg: origin xyz=-0.22 0 .25 -> xyz=0 0.22 0.25
- joint base_to_right_leg: origin xyz=0.22 0 .25 -> xyz=0 -0.22 0.25

File: urdf/05-visual.urdf (robot description, URDF)
Before this commit: robot visual, 16 links, 15 joints
Links:
- link box: geometry visual box size=0.08 0.08 0.08
- link gripper_pole: geometry visual cylinder length=0.2 radius=0.01
- link left_back_wheel: geometry visual cylinder length=0.1 radius=0.035
- link left_base: geometry visual box size=0.4 0.1 0.1
- link left_front_wheel: geometry visual cylinder length=0.1 radius=0.035
- link left_gripper: geometry visual mesh filename=package://urdf_tutorial/meshes/l_finger.dae
- link left_leg: geometry visual box size=0.6 0.1 0.2
- link left_tip: geometry visual mesh filename=package://urdf_tutorial/meshes/l_finger_tip.dae
- link right_back_wheel: geometry visual cylinder length=0.1 radius=0.035
- link right_base: geometry visual box size=0.4 0.1 0.1
- link right_front_wheel: geometry visual cylinder length=0.1 radius=0.035
- link right_gripper: geometry visual mesh filename=package://urdf_tutorial/meshes/l_finger.dae
- link right_leg: geometry visual box size=0.6 0.1 0.2
- link right_tip: geometry visual mesh filename=package://urdf_tutorial/meshes/l_finger_tip.dae
Joints:
- joint base_to_left_leg: origin xyz=-0.22 0 .25 -> xyz=0 0.22 0.25
- joint base_to_right_leg: origin xyz=0.22 0 .25 -> xyz=0 -0.22 0.25
- joint gripper_extension: origin xyz=0 0.19 .2 rpy=0 0 1.57075 -> xyz=0.19 0 0.2 rpy=0 0 0
- joint left_back_wheel_joint: origin xyz=0 -0.133333333333 -0.085 rpy=0 1.57075 0 -> xyz=-0.133333333333 0 -0.085 rpy=0 0 0
- joint left_front_wheel_joint: origin xyz=0 0.133333333333 -0.085 rpy=0 1.57075 0 -> xyz=0.133333333333 0 -0.085 rpy=0 0 0
- joint right_back_wheel_joint: origin xyz=0 -0.133333333333 -0.085 rpy=0 1.57075 0 -> xyz=-0.133333333333 0 -0.085 rpy=0 0 0
- joint right_front_wheel_joint: origin xyz=0 0.133333333333 -0.085 rpy=0 1.57075 0 -> xyz=0.133333333333 0 -0.085 rpy=0 0 0
- joint tobox: origin xyz=0 0.1414 0.1414 -> xyz=0.1814 0 0.1414

File: urdf/06-flexible.urdf (robot description, URDF)
Before this commit: robot flexible, 16 links, 15 joints
Links:
- link box: geometry visual box size=0.08 0.08 0.08
- link gripper_pole: geometry visual cylinder length=0.2 radius=0.01
- link left_back_wheel: geometry visual cylinder length=0.1 radius=0.035
- link left_base: geometry visual box size=0.4 0.1 0.1
- link left_front_wheel: geometry visual cylinder length=0.1 radius=0.035
- link left_gripper: geometry visual mesh filename=package://urdf_tutorial/meshes/l_finger.dae
- link left_leg: geometry visual box size=0.6 0.1 0.2
- link left_tip: geometry visual mesh filename=package://urdf_tutorial/meshes/l_finger_tip.dae
- link right_back_wheel: geometry visual cylinder length=0.1 radius=0.035
- link right_base: geometry visual box size=0.4 0.1 0.1
- link right_front_wheel: geometry visual cylinder length=0.1 radius=0.035
- link right_gripper: geometry visual mesh filename=package://urdf_tutorial/meshes/l_finger.dae
- link right_leg: geometry visual box size=0.6 0.1 0.2
- link right_tip: geometry visual mesh filename=package://urdf_tutorial/meshes/l_finger_tip.dae
Joints:
- joint base_to_left_leg: origin xyz=-0.22 0 .25 -> xyz=0 0.22 0.25
- joint base_to_right_leg: origin xyz=0.22 0 .25 -> xyz=0 -0.22 0.25
- joint gripper_extension: origin xyz=0 0.19 .2 rpy=0 0 1.57075 -> xyz=0.19 0 0.2 rpy=0 0 0
- joint left_back_wheel_joint: axis 0 0 1 -> 0 1 0; limit effort=100 velocity=100 -> (none); origin xyz=0 -0.133333333333 -0.085 rpy=0 1.57075 0 -> xyz=-0.133333333333 0 -0.085 rpy=0 0 0
- joint left_front_wheel_joint: axis 0 0 1 -> 0 1 0; limit effort=100 velocity=100 -> (none); origin xyz=0 0.133333333333 -0.085 rpy=0 1.57075 0 -> xyz=0.133333333333 0 -0.085 rpy=0 0 0
- joint right_back_wheel_joint: axis 0 0 1 -> 0 1 0; limit effort=100 velocity=100 -> (none); origin xyz=0 -0.133333333333 -0.085 rpy=0 1.57075 0 -> xyz=-0.133333333333 0 -0.085 rpy=0 0 0
- joint right_front_wheel_joint: axis 0 0 1 -> 0 1 0; limit effort=100 velocity=100 -> (none); origin xyz=0 0.133333333333 -0.085 rpy=0 1.57075 0 -> xyz=0.133333333333 0 -0.085 rpy=0 0 0
- joint tobox: origin xyz=0 0.1414 0.1414 -> xyz=0.1814 0 0.1414

File: urdf/07-physics.urdf (robot description, URDF)
Before this commit: robot physics, 16 links, 15 joints
Links:
- link box: geometry collision box size=0.08 0.08 0.08; visual box size=0.08 0.08 0.08
- link gripper_pole: geometry collision cylinder length=0.2 radius=0.01; visual cylinder length=0.2 radius=0.01
- link head: mass 10 -> 2
- link left_back_wheel: geometry collision cylinder length=0.1 radius=0.035; visual cylinder length=0.1 radius=0.035
- link left_base: geometry collision box size=0.4 0.1 0.1; visual box size=0.4 0.1 0.1
- link left_front_wheel: geometry collision cylinder length=0.1 radius=0.035; visual cylinder length=0.1 radius=0.035
- link left_gripper: geometry collision mesh filename=package://urdf_tutorial/meshes/l_finger.dae; visual mesh filename=package://urdf_tutorial/meshes/l_finger.dae
- link left_leg: geometry collision box size=0.6 0.1 0.2; visual box size=0.6 0.1 0.2
- link left_tip: geometry collision mesh filename=package://urdf_tutorial/meshes/l_finger_tip.dae; visual mesh filename=package://urdf_tutorial/meshes/l_finger_tip.dae
- link right_back_wheel: geometry collision cylinder length=0.1 radius=0.035; visual cylinder length=0.1 radius=0.035
- link right_base: geometry collision box size=0.4 0.1 0.1; visual box size=0.4 0.1 0.1
- link right_front_wheel: geometry collision cylinder length=0.1 radius=0.035; visual cylinder length=0.1 radius=0.035
- link right_gripper: geometry collision mesh filename=package://urdf_tutorial/meshes/l_finger.dae; visual mesh filename=package://urdf_tutorial/meshes/l_finger.dae
- link right_leg: geometry collision box size=0.6 0.1 0.2; visual box size=0.6 0.1 0.2
- link right_tip: geometry collision mesh filename=package://urdf_tutorial/meshes/l_finger_tip.dae; visual mesh filename=package://urdf_tutorial/meshes/l_finger_tip.dae
Joints:
- joint base_to_left_leg: origin xyz=-0.22 0 .25 -> xyz=0 0.22 0.25
- joint base_to_right_leg: origin xyz=0.22 0 .25 -> xyz=0 -0.22 0.25
- joint gripper_extension: origin xyz=0 0.19 .2 rpy=0 0 1.57075 -> xyz=0.19 0 0.2 rpy=0 0 0
- joint left_back_wheel_joint: axis 0 0 1 -> 0 1 0; limit effort=100 velocity=100 -> (none); origin xyz=0 -0.133333333333 -0.085 rpy=0 1.57075 0 -> xyz=-0.133333333333 0 -0.085 rpy=0 0 0
- joint left_front_wheel_joint: axis 0 0 1 -> 0 1 0; limit effort=100 velocity=100 -> (none); origin xyz=0 0.133333333333 -0.085 rpy=0 1.57075 0 -> xyz=0.133333333333 0 -0.085 rpy=0 0 0
- joint right_back_wheel_joint: axis 0 0 1 -> 0 1 0; limit effort=100 velocity=100 -> (none); origin xyz=0 -0.133333333333 -0.085 rpy=0 1.57075 0 -> xyz=-0.133333333333 0 -0.085 rpy=0 0 0
- joint right_front_wheel_joint: axis 0 0 1 -> 0 1 0; limit effort=100 velocity=100 -> (none); origin xyz=0 0.133333333333 -0.085 rpy=0 1.57075 0 -> xyz=0.133333333333 0 -0.085 rpy=0 0 0
- joint tobox: origin xyz=0 0.1414 0.1414 -> xyz=0.1814 0 0.1414

File: urdf/08-macroed.urdf.xacro (robot description, xacro)
@@ -1,216 +1,215 @@
 <?xml version="1.0"?>
-<robot xmlns:sensor="http://playerstage.sourceforge.net/gazebo/xmlschema/#sensor"
-	 xmlns:controller="http://playerstage.sourceforge.net/gazebo/xmlschema/#controller"
-	 xmlns:interface="http://playerstage.sourceforge.net/gazebo/xmlschema/#interface"
-	 xmlns:xacro="http://playerstage.sourceforge.net/gazebo/xmlschema/#interface" name="macroed">
-	<xacro:property name="width" value=".2" />
-	<xacro:property name="leglen" value=".6" />
-	<xacro:property name="polelen" value=".2" />
-	<xacro:property name="bodylen" value=".6" />
-	<xacro:property name="baselen" value=".4" />
-	<xacro:property name="wheeldiam" value=".07" />
-	<xacro:property name="pi" value="3.1415" />
-	<xacro:macro name="default_inertial" params="mass">
-		<inertial>
-      			<mass value="${mass}" />
-		        <inertia ixx="1.0" ixy="0.0" ixz="0.0"
-			         iyy="1.0" iyz="0.0"
-			         izz="1.0" />
-		</inertial>
-	</xacro:macro>
-	<link name="base_link">
-		<visual>
-			<geometry>
-				<cylinder radius="${width}" length="${bodylen}"/>
-			</geometry>
-			<material name="blue">
-				<color rgba="0 0 .8 1"/>
-			</material>
-		</visual>
-		<collision>
-			<geometry>
-				<cylinder radius="${width}" length="${bodylen}"/>
-			</geometry>
-		</collision>
-		<xacro:default_inertial mass="10"/>
-	</link>
-	<xacro:macro name="wheel" params="prefix suffix reflect">
-		<link name="${prefix}_${suffix}_wheel">
-			<visual>
-				<geometry>
-					<cylinder radius="${wheeldiam/2}" length=".1"/>
-				</geometry>
-				<material name="black">
-					<color rgba="0 0 0 1"/>
-				</material>
-			</visual>
-			<collision>
-				<geometry>
-					<cylinder radius="${wheeldiam/2}" length=".1"/>
-				</geometry>
-			</collision>
-			<xacro:default_inertial mass="1"/>
-		</link>
-		<joint name="${prefix}_${suffix}_wheel_joint" type="continuous">
-			<axis xyz="0 0 1"/>
-			<parent link="${prefix}_base"/>
-			<child link="${prefix}_${suffix}_wheel"/>
-			<origin xyz="0 ${baselen*reflect/3} -${wheeldiam/2+.05}" rpy="0 ${pi/2} 0"/>
-      			<limit effort="100" velocity="100" />
-			<joint_properties damping="0.0" friction="0.0" />
-		</joint>
-	</xacro:macro>
-	<xacro:macro name="leg" params="prefix reflect">
-		<link name="${prefix}_leg">
-			<visual>
-				<geometry>
-					<box size="${leglen} .2 .1"/>
-				</geometry>
-				<origin xyz="0 0 -${leglen/2}" rpy="0 ${pi/2} 0"/>
-				<material name="white">
-					<color rgba="1 1 1 1"/>
-				</material>
-			</visual>
-			<collision>
-				<geometry>
-					<box size="${leglen} .2 .1"/>
-				</geometry>
-				<origin xyz="0 0 -${leglen/2}" rpy="0 ${pi/2} 0"/>
-			</collision>
-			<xacro:default_inertial mass="10"/>
-		</link>
-		<joint name="base_to_${prefix}_leg" type="fixed">
-			<parent link="base_link"/>
-			<child link="${prefix}_leg"/>
-			<origin xyz="${reflect*(width+.02)} 0 .25" />
-		</joint>
-		<link name="${prefix}_base">
-			<visual>
-				<geometry>
-					<box size=".1 ${baselen} .1"/>
-				</geometry>
-				<material name="white"/>
-			</visual>
-			<collision>
-				<geometry>
-					<box size=".1 ${baselen} .1"/>
-				</geometry>
-			</collision>
-			<xacro:default_inertial mass="10"/>
-		</link>
-		<joint name="${prefix}_base_joint" type="fixed">
-			<parent link="${prefix}_leg"/>
-			<child link="${prefix}_base"/>
-			<origin xyz="0 0 ${-leglen}" />
-		</joint>
-		<xacro:wheel prefix="${prefix}" suffix="front" reflect="1"/>
-		<xacro:wheel prefix="${prefix}" suffix="back" reflect="-1"/>
-	</xacro:macro>
-	<xacro:leg prefix="right" reflect="1" />
-	<xacro:leg prefix="left" reflect="-1" />
-	<joint name="gripper_extension" type="prismatic">
-		<parent link="base_link"/>
-		<child link="gripper_pole"/>
-    		<limit effort="1000.0" lower="-${width*2-.02}" upper="0" velocity="0.5"/>
-		<origin rpy="0 0 ${pi/2}" xyz="0 ${width-.01} .2"/>
-	</joint>
-	<link name="gripper_pole">
-		<visual>
-			<geometry>
-				<cylinder length="${polelen}" radius=".01"/>
-			</geometry>
-			<origin xyz="${polelen/2} 0 0" rpy="0 ${pi/2} 0 "/>
-		</visual>
-		<collision>
-			<geometry>
-				<cylinder length="${polelen}" radius=".01"/>
-			</geometry>
-			<origin xyz="${polelen/2} 0 0" rpy="0 ${pi/2} 0 "/>
-		</collision>
-		<xacro:default_inertial mass=".05"/>
-	</link>
-	<xacro:macro name="gripper" params="prefix reflect">
-		<joint name="${prefix}_gripper_joint" type="revolute">
-			<axis xyz="0 0 ${reflect}"/>
-			<limit effort="1000.0" lower="0.0" upper="0.548" velocity="0.5"/>
-			<origin rpy="0 0 0" xyz="${polelen} ${reflect*0.01} 0"/>
-			<parent link="gripper_pole"/>
-			<child link="${prefix}_gripper"/>
-		</joint>
-		<link name="${prefix}_gripper">
-			<visual>
-     				<origin rpy="${(reflect-1)/2*pi} 0 0" xyz="0 0 0"/>
-				<geometry>
-					<mesh filename="package://pr2_description/meshes/gripper_v0/l_finger.dae"/>
-				</geometry>
-			</visual>
-			<collision>
-				<geometry>
-					<mesh filename="package://pr2_description/meshes/gripper_v0/l_finger.dae"/>
-				</geometry>
-     				<origin rpy="${(reflect-1)/2*pi} 0 0" xyz="0 0 0"/>
-			</collision>
-			<xacro:default_inertial mass=".05"/>
-		</link>
-		<joint name="${prefix}_tip_joint" type="fixed">
-			<parent link="${prefix}_gripper"/>
-			<child link="${prefix}_tip"/>
-		</joint>
-		<link name="${prefix}_tip">
-			<visual>
-     				<origin rpy="${(reflect-1)/2*pi} 0 0" xyz="0.09137 0.00495 0"/>
-				<geometry>
-					<mesh filename="package://pr2_description/meshes/gripper_v0/l_finger_tip.dae"/>
-				</geometry>
-			</visual>
-			<collision>
-				<geometry>
-					<mesh filename="package://pr2_description/meshes/gripper_v0/l_finger_tip.dae"/>
-				</geometry>
-     				<origin rpy="${(reflect-1)/2*pi} 0 0" xyz="0.09137 0.00495 0"/>
-			</collision>
-			<xacro:default_inertial mass=".05"/>
-		</link>
-	</xacro:macro>
-	<xacro:gripper prefix="left" reflect="1" />
-	<xacro:gripper prefix="right" reflect="-1" />
-	<link name="head">
-		<visual>
-			<geometry>
-				<sphere radius="${width}"/>
-			</geometry>
-			<material name="white"/>
-		</visual>
-		<collision>
-			<geometry>
-				<sphere radius="${width}"/>
-			</geometry>
-		</collision>
-		<xacro:default_inertial mass="10"/>
-	</link>
-	<joint name="head_swivel" type="continuous">
-		<parent link="base_link"/>
-		<child link="head"/>
-		<axis xyz="0 0 1"/>
-		<origin xyz="0 0 ${bodylen/2}"/>
-	</joint>
-	<link name="box">
-		<visual>
-			<geometry>
-				<box size=".08 .08 .08"/>
-			</geometry>
-			<material name="blue"/>
-		</visual>
-		<collision>
-			<geometry>
-				<box size=".08 .08 .08"/>
-			</geometry>
-		</collision>
-		<xacro:default_inertial mass="1"/>
-	</link>
-	<joint name="tobox" type="fixed">
-		<parent link="head"/>
-		<child link="box"/>
-		<origin xyz="0 ${.707*width} ${.707*width}"/>
-	</joint>
+<robot name="macroed" xmlns:xacro="http://ros.org/wiki/xacro">
+  <xacro:property name="width" value="0.2" />
+  <xacro:property name="leglen" value="0.6" />
+  <xacro:property name="polelen" value="0.2" />
+  <xacro:property name="bodylen" value="0.6" />
+  <xacro:property name="baselen" value="0.4" />
+  <xacro:property name="wheeldiam" value="0.07" />
+  <xacro:property name="pi" value="3.1415" />
+  <material name="blue">
+    <color rgba="0 0 0.8 1"/>
+  </material>
+  <material name="black">
+    <color rgba="0 0 0 1"/>
+  </material>
+  <material name="white">
+    <color rgba="1 1 1 1"/>
+  </material>
+  <xacro:macro name="default_inertial" params="mass">
+    <inertial>
+      <mass value="${mass}" />
+      <inertia ixx="1.0" ixy="0.0" ixz="0.0" iyy="1.0" iyz="0.0" izz="1.0" />
+    </inertial>
+  </xacro:macro>
+  <link name="base_link">
+    <visual>
+      <geometry>
+        <cylinder radius="${width}" length="${bodylen}"/>
+      </geometry>
+      <material name="blue"/>
+    </visual>
+    <collision>
+      <geometry>
+        <cylinder radius="${width}" length="${bodylen}"/>
+      </geometry>
+    </collision>
+    <xacro:default_inertial mass="10"/>
+  </link>
+  <xacro:macro name="wheel" params="prefix suffix reflect">
+    <link name="${prefix}_${suffix}_wheel">
+      <visual>
+        <origin xyz="0 0 0" rpy="${pi/2} 0 0" />
+        <geometry>
+          <cylinder radius="${wheeldiam/2}" length="0.1"/>
+        </geometry>
+        <material name="black"/>
+      </visual>
+      <collision>
+        <origin xyz="0 0 0" rpy="${pi/2} 0 0" />
+        <geometry>
+          <cylinder radius="${wheeldiam/2}" length="0.1"/>
+        </geometry>
+      </collision>
+      <xacro:default_inertial mass="1"/>
+    </link>
+    <joint name="${prefix}_${suffix}_wheel_joint" type="continuous">
+      <axis xyz="0 1 0" rpy="0 0 0" />
+      <parent link="${prefix}_base"/>
+      <child link="${prefix}_${suffix}_wheel"/>
+      <origin xyz="${baselen*reflect/3} 0 -${wheeldiam/2+.05}" rpy="0 0 0"/>
+    </joint>
+  </xacro:macro>
+  <xacro:macro name="leg" params="prefix reflect">
+    <link name="${prefix}_leg">
+      <visual>
+        <geometry>
+          <box size="${leglen} 0.1 0.2"/>
+        </geometry>
+        <origin xyz="0 0 -${leglen/2}" rpy="0 ${pi/2} 0"/>
+        <material name="white"/>
+      </visual>
+      <collision>
+        <geometry>
+          <box size="${leglen} 0.1 0.2"/>
+        </geometry>
+        <origin xyz="0 0 -${leglen/2}" rpy="0 ${pi/2} 0"/>
+      </collision>
+      <xacro:default_inertial mass="10"/>
+    </link>
+    <joint name="base_to_${prefix}_leg" type="fixed">
+      <parent link="base_link"/>
+      <child link="${prefix}_leg"/>
+      <origin xyz="0 ${reflect*(width+.02)} 0.25" />
+    </joint>
+    <link name="${prefix}_base">
+      <visual>
+        <geometry>
+          <box size="${baselen} 0.1 0.1"/>
+        </geometry>
+        <material name="white"/>
+      </visual>
+      <collision>
+        <geometry>
+          <box size="${baselen} 0.1 0.1"/>
+        </geometry>
+      </collision>
+      <xacro:default_inertial mass="10"/>
+    </link>
+    <joint name="${prefix}_base_joint" type="fixed">
+      <parent link="${prefix}_leg"/>
+      <child link="${prefix}_base"/>
+      <origin xyz="0 0 ${-leglen}" />
+    </joint>
+    <xacro:wheel prefix="${prefix}" suffix="front" reflect="1"/>
+    <xacro:wheel prefix="${prefix}" suffix="back" reflect="-1"/>
+  </xacro:macro>
+  <xacro:leg prefix="right" reflect="-1" />
+  <xacro:leg prefix="left" reflect="1" />
+  <joint name="gripper_extension" type="prismatic">
+    <parent link="base_link"/>
+    <child link="gripper_pole"/>
+    <limit effort="1000.0" lower="-${width*2-.02}" upper="0" velocity="0.5"/>
+    <origin rpy="0 0 0" xyz="${width-.01} 0 0.2"/>
+  </joint>
+  <link name="gripper_pole">
+    <visual>
+      <geometry>
+        <cylinder length="${polelen}" radius="0.01"/>
+      </geometry>
+      <origin xyz="${polelen/2} 0 0" rpy="0 ${pi/2} 0 "/>
+    </visual>
+    <collision>
+      <geometry>
+        <cylinder length="${polelen}" radius="0.01"/>
+      </geometry>
+      <origin xyz="${polelen/2} 0 0" rpy="0 ${pi/2} 0 "/>
+    </collision>
+    <xacro:default_inertial mass="0.05"/>
+  </link>
+  <xacro:macro name="gripper" params="prefix reflect">
+    <joint name="${prefix}_gripper_joint" type="revolute">
+      <axis xyz="0 0 ${reflect}"/>
+      <limit effort="1000.0" lower="0.0" upper="0.548" velocity="0.5"/>
+      <origin rpy="0 0 0" xyz="${polelen} ${reflect*0.01} 0"/>
+      <parent link="gripper_pole"/>
+      <child link="${prefix}_gripper"/>
+    </joint>
+    <link name="${prefix}_gripper">
+      <visual>
+        <origin rpy="${(reflect-1)/2*pi} 0 0" xyz="0 0 0"/>
+        <geometry>
+          <mesh filename="package://urdf_tutorial/meshes/l_finger.dae"/>
+        </geometry>
+      </visual>
+      <collision>
+        <geometry>
+          <mesh filename="package://urdf_tutorial/meshes/l_finger.dae"/>
+        </geometry>
+        <origin rpy="${(reflect-1)/2*pi} 0 0" xyz="0 0 0"/>
+      </collision>
+      <xacro:default_inertial mass="0.05"/>
+    </link>
+    <joint name="${prefix}_tip_joint" type="fixed">
+      <parent link="${prefix}_gripper"/>
+      <child link="${prefix}_tip"/>
+    </joint>
+    <link name="${prefix}_tip">
+      <visual>
+        <origin rpy="${(reflect-1)/2*pi} 0 0" xyz="0.09137 0.00495 0"/>
+        <geometry>
+          <mesh filename="package://urdf_tutorial/meshes/l_finger_tip.dae"/>
+        </geometry>
+      </visual>
+      <collision>
+        <geometry>
+          <mesh filename="package://urdf_tutorial/meshes/l_finger_tip.dae"/>
+        </geometry>
+        <origin rpy="${(reflect-1)/2*pi} 0 0" xyz="0.09137 0.00495 0"/>
+      </collision>
+      <xacro:default_inertial mass="0.05"/>
+    </link>
+  </xacro:macro>
+  <xacro:gripper prefix="left" reflect="1" />
+  <xacro:gripper prefix="right" reflect="-1" />
+  <link name="head">
+    <visual>
+      <geometry>
+        <sphere radius="${width}"/>
+      </geometry>
+      <material name="white"/>
+    </visual>
+    <collision>
+      <geometry>
+        <sphere radius="${width}"/>
+      </geometry>
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
File: urdf/09-roscontrol.urdf.xacro (robot description, xacro)
@@ -1,4 +1,4 @@
 <?xml version="1.0"?>
-<robot name="r2d2" xmlns:xacro="http://ros.org/wiki/xacro">
+<robot name="roscontrol" xmlns:xacro="http://ros.org/wiki/xacro">
   <xacro:property name="width" value="0.2" />
   <xacro:property name="leglen" value="0.6" />
