Commit message: Imported upstream version '0.3.0' of 'upstream'

File: urdf_sim_tutorial/urdf/09-publishjoints.urdf.xacro (robot description, xacro)
@@ -1,4 +1,4 @@
 <?xml version="1.0"?>
-<robot name="roscontrol" xmlns:xacro="http://ros.org/wiki/xacro">
+<robot name="gazebo1" xmlns:xacro="http://ros.org/wiki/xacro">
   <xacro:property name="width" value="0.2" />
   <xacro:property name="leglen" value="0.6" />
@@ -45,5 +45,4 @@
         </geometry>
         <material name="black"/>
-        <origin xyz="0 0 0" rpy="0 0 0" />
       </visual>
       <collision>
@@ -52,5 +51,4 @@
           <cylinder radius="${wheeldiam/2}" length="0.1"/>
         </geometry>
-        <origin xyz="0 0 0" rpy="0 0 0" />
       </collision>
       <xacro:default_inertial mass="1"/>
@@ -62,24 +60,4 @@
       <origin xyz="${baselen*reflect/3} 0 -${wheeldiam/2+.05}" rpy="0 0 0"/>
     </joint>
-    <!-- This block provides the simulator (Gazebo) with information on a few additional
-    physical properties. See http://gazebosim.org/tutorials/?tut=ros_urdf for more-->
-    <gazebo reference="${prefix}_${suffix}_wheel">
-      <mu1 value="200.0"/>
-      <mu2 value="100.0"/>
-      <kp value="10000000.0" />
-      <kd value="1.0" />
-      <material>Gazebo/Grey</material>
-    </gazebo>
-    <!-- This block connects the wheel joint to an actuator (motor), which informs both
-    simulation and visualization of the robot -->
-    <transmission name="${prefix}_${suffix}_wheel_trans" type="SimpleTransmission">
-      <type>transmission_interface/SimpleTransmission</type>
-      <actuator name="${prefix}_${suffix}_wheel_motor">
-        <mechanicalReduction>1</mechanicalReduction>
-      </actuator>
-      <joint name="${prefix}_${suffix}_wheel_joint">
-        <hardwareInterface>VelocityJointInterface</hardwareInterface>
-      </joint>
-    </transmission>
   </xacro:macro>
   <xacro:macro name="leg" params="prefix reflect">
@@ -134,6 +112,4 @@
     <limit effort="1000.0" lower="-${width*2-.02}" upper="0" velocity="0.5"/>
     <origin rpy="0 0 0" xyz="${width-.01} 0 0.2"/>
-    <limit effort="30" velocity="0.2"/>
-    <dynamics damping="0.0" friction="0.0"/>
   </joint>
   <link name="gripper_pole">
@@ -152,13 +128,4 @@
     <xacro:default_inertial mass="0.05"/>
   </link>
-  <transmission name="gripper_extension_trans" type="SimpleTransmission">
-    <type>transmission_interface/SimpleTransmission</type>
-    <actuator name="gripper_extension_motor">
-      <mechanicalReduction>1</mechanicalReduction>
-    </actuator>
-    <joint name="gripper_extension">
-      <hardwareInterface>PositionJointInterface</hardwareInterface>
-    </joint>
-  </transmission>
   <xacro:macro name="gripper" params="prefix reflect">
     <joint name="${prefix}_gripper_joint" type="revolute">
@@ -168,6 +135,4 @@
       <parent link="gripper_pole"/>
       <child link="${prefix}_gripper"/>
-      <limit effort="30" velocity="1.0"/>
-      <dynamics damping="0.0" friction="0.0"/>
     </joint>
     <link name="${prefix}_gripper">
@@ -186,13 +151,4 @@
       <xacro:default_inertial mass="0.05"/>
     </link>
-    <transmission name="${prefix}_gripper_trans" type="SimpleTransmission">
-      <type>transmission_interface/SimpleTransmission</type>
-      <actuator name="${prefix}_gripper_motor">
-        <mechanicalReduction>1</mechanicalReduction>
-      </actuator>
-      <joint name="${prefix}_gripper_joint">
-        <hardwareInterface>PositionJointInterface</hardwareInterface>
-      </joint>
-    </transmission>
     <joint name="${prefix}_tip_joint" type="fixed">
       <parent link="${prefix}_gripper"/>
@@ -236,18 +192,5 @@
     <axis xyz="0 0 1"/>
     <origin xyz="0 0 ${bodylen/2}"/>
-    <limit effort="30" velocity="1.0"/>
-    <dynamics damping="0.0" friction="0.0"/>
   </joint>
-  <!-- This block connects the head_swivel joint to an actuator (motor), which informs both
-  simulation and visualization of the robot -->
-  <transmission name="head_swivel_trans" type="SimpleTransmission">
-    <type>transmission_interface/SimpleTransmission</type>
-    <actuator name="$head_swivel_motor">
-      <mechanicalReduction>1</mechanicalReduction>
-    </actuator>
-    <joint name="head_swivel">
-      <hardwareInterface>PositionJointInterface</hardwareInterface>
-    </joint>
-  </transmission>
   <link name="box">
     <visual>

File: urdf_sim_tutorial/urdf/10-firsttransmission.urdf.xacro (robot description, xacro)
@@ -1,4 +1,4 @@
 <?xml version="1.0"?>
-<robot name="r2d2" xmlns:xacro="http://ros.org/wiki/xacro">
+<robot name="first_transmission" xmlns:xacro="http://ros.org/wiki/xacro">
   <xacro:property name="width" value="0.2" />
   <xacro:property name="leglen" value="0.6" />
@@ -45,5 +45,4 @@
         </geometry>
         <material name="black"/>
-        <origin xyz="0 0 0" rpy="0 0 0" />
       </visual>
       <collision>
@@ -52,5 +51,4 @@
           <cylinder radius="${wheeldiam/2}" length="0.1"/>
         </geometry>
-        <origin xyz="0 0 0" rpy="0 0 0" />
       </collision>
       <xacro:default_inertial mass="1"/>
@@ -62,24 +60,4 @@
       <origin xyz="${baselen*reflect/3} 0 -${wheeldiam/2+.05}" rpy="0 0 0"/>
     </joint>
-    <!-- This block provides the simulator (Gazebo) with information on a few additional
-    physical properties. See http://gazebosim.org/tutorials/?tut=ros_urdf for more-->
-    <gazebo reference="${prefix}_${suffix}_wheel">
-      <mu1 value="200.0"/>
-      <mu2 value="100.0"/>
-      <kp value="10000000.0" />
-      <kd value="1.0" />
-      <material>Gazebo/Grey</material>
-    </gazebo>
-    <!-- This block connects the wheel joint to an actuator (motor), which informs both
-    simulation and visualization of the robot -->
-    <transmission name="${prefix}_${suffix}_wheel_trans" type="SimpleTransmission">
-      <type>transmission_interface/SimpleTransmission</type>
-      <actuator name="${prefix}_${suffix}_wheel_motor">
-        <mechanicalReduction>1</mechanicalReduction>
-      </actuator>
-      <joint name="${prefix}_${suffix}_wheel_joint">
-        <hardwareInterface>VelocityJointInterface</hardwareInterface>
-      </joint>
-    </transmission>
   </xacro:macro>
   <xacro:macro name="leg" params="prefix reflect">
@@ -134,6 +112,4 @@
     <limit effort="1000.0" lower="-${width*2-.02}" upper="0" velocity="0.5"/>
     <origin rpy="0 0 0" xyz="${width-.01} 0 0.2"/>
-    <limit effort="30" velocity="0.2"/>
-    <dynamics damping="0.0" friction="0.0"/>
   </joint>
   <link name="gripper_pole">
@@ -152,13 +128,4 @@
     <xacro:default_inertial mass="0.05"/>
   </link>
-  <transmission name="gripper_extension_trans" type="SimpleTransmission">
-    <type>transmission_interface/SimpleTransmission</type>
-    <actuator name="gripper_extension_motor">
-      <mechanicalReduction>1</mechanicalReduction>
-    </actuator>
-    <joint name="gripper_extension">
-      <hardwareInterface>PositionJointInterface</hardwareInterface>
-    </joint>
-  </transmission>
   <xacro:macro name="gripper" params="prefix reflect">
     <joint name="${prefix}_gripper_joint" type="revolute">
@@ -168,6 +135,4 @@
       <parent link="gripper_pole"/>
       <child link="${prefix}_gripper"/>
-      <limit effort="30" velocity="1.0"/>
-      <dynamics damping="0.0" friction="0.0"/>
     </joint>
     <link name="${prefix}_gripper">
@@ -186,13 +151,4 @@
       <xacro:default_inertial mass="0.05"/>
     </link>
-    <transmission name="${prefix}_gripper_trans" type="SimpleTransmission">
-      <type>transmission_interface/SimpleTransmission</type>
-      <actuator name="${prefix}_gripper_motor">
-        <mechanicalReduction>1</mechanicalReduction>
-      </actuator>
-      <joint name="${prefix}_gripper_joint">
-        <hardwareInterface>PositionJointInterface</hardwareInterface>
-      </joint>
-    </transmission>
     <joint name="${prefix}_tip_joint" type="fixed">
       <parent link="${prefix}_gripper"/>
@@ -236,10 +192,8 @@
     <axis xyz="0 0 1"/>
     <origin xyz="0 0 ${bodylen/2}"/>
-    <limit effort="30" velocity="1.0"/>
-    <dynamics damping="0.0" friction="0.0"/>
   </joint>
   <!-- This block connects the head_swivel joint to an actuator (motor), which informs both
   simulation and visualization of the robot -->
-  <transmission name="head_swivel_trans" type="SimpleTransmission">
+  <transmission name="head_swivel_trans">
     <type>transmission_interface/SimpleTransmission</type>
     <actuator name="$head_swivel_motor">

File: urdf_sim_tutorial/urdf/12-gripper.urdf.xacro (robot description, xacro)
@@ -1,4 +1,4 @@
 <?xml version="1.0"?>
-<robot name="macroed" xmlns:xacro="http://ros.org/wiki/xacro">
+<robot name="r2d2" xmlns:xacro="http://ros.org/wiki/xacro">
   <xacro:property name="width" value="0.2" />
   <xacro:property name="leglen" value="0.6" />
@@ -112,4 +112,6 @@
     <limit effort="1000.0" lower="-${width*2-.02}" upper="0" velocity="0.5"/>
     <origin rpy="0 0 0" xyz="${width-.01} 0 0.2"/>
+    <limit effort="30" velocity="0.2"/>
+    <dynamics damping="0.0" friction="0.0"/>
   </joint>
   <link name="gripper_pole">
@@ -128,4 +130,13 @@
     <xacro:default_inertial mass="0.05"/>
   </link>
+  <transmission name="gripper_extension_trans" type="SimpleTransmission">
+    <type>transmission_interface/SimpleTransmission</type>
+    <actuator name="gripper_extension_motor">
+      <mechanicalReduction>1</mechanicalReduction>
+    </actuator>
+    <joint name="gripper_extension">
+      <hardwareInterface>PositionJointInterface</hardwareInterface>
+    </joint>
+  </transmission>
   <xacro:macro name="gripper" params="prefix reflect">
     <joint name="${prefix}_gripper_joint" type="revolute">
@@ -135,4 +146,6 @@
       <parent link="gripper_pole"/>
       <child link="${prefix}_gripper"/>
+      <limit effort="30" velocity="1.0"/>
+      <dynamics damping="0.0" friction="0.0"/>
     </joint>
     <link name="${prefix}_gripper">
@@ -151,4 +164,13 @@
       <xacro:default_inertial mass="0.05"/>
     </link>
+    <transmission name="${prefix}_gripper_trans" type="SimpleTransmission">
+      <type>transmission_interface/SimpleTransmission</type>
+      <actuator name="${prefix}_gripper_motor">
+        <mechanicalReduction>1</mechanicalReduction>
+      </actuator>
+      <joint name="${prefix}_gripper_joint">
+        <hardwareInterface>PositionJointInterface</hardwareInterface>
+      </joint>
+    </transmission>
     <joint name="${prefix}_tip_joint" type="fixed">
       <parent link="${prefix}_gripper"/>
@@ -192,5 +214,18 @@
     <axis xyz="0 0 1"/>
     <origin xyz="0 0 ${bodylen/2}"/>
+    <limit effort="30" velocity="1.0"/>
+    <dynamics damping="0.0" friction="0.0"/>
   </joint>
+  <!-- This block connects the head_swivel joint to an actuator (motor), which informs both
+  simulation and visualization of the robot -->
+  <transmission name="head_swivel_trans">
+    <type>transmission_interface/SimpleTransmission</type>
+    <actuator name="$head_swivel_motor">
+      <mechanicalReduction>1</mechanicalReduction>
+    </actuator>
+    <joint name="head_swivel">
+      <hardwareInterface>PositionJointInterface</hardwareInterface>
+    </joint>
+  </transmission>
   <link name="box">
     <visual>
@@ -213,3 +248,9 @@
     <origin xyz="${.707*width+0.04} 0 ${.707*width}"/>
   </joint>
+  <!-- Gazebo plugin for ROS Control -->
+  <gazebo>
+    <plugin name="gazebo_ros_control" filename="libgazebo_ros_control.so">
+      <robotNamespace>/</robotNamespace>
+    </plugin>
+  </gazebo>
 </robot>
